Commit message: Try to get the unit tests to pass.

File: test/sphere_wheel.xacro (robot description, xacro)
@@ -1,5 +1,5 @@
 <?xml version="1.0"?>
 <robot xmlns:xacro="http://www.ros.org/wiki/xacro">
-  <macro name="sphere_wheel" params="name parent radius *origin">
+  <xacro:macro name="sphere_wheel" params="name parent radius *origin">
     <link name="${name}_link">
       <inertial>
@@ -37,4 +37,4 @@
       <material>Gazebo/Red</material>
     </gazebo>
-  </macro>
+  </xacro:macro>
 </robot>

File: test/wheel.xacro (robot description, xacro)
@@ -1,5 +1,5 @@
 <?xml version="1.0"?>
 <robot xmlns:xacro="http://www.ros.org/wiki/xacro">
-  <macro name="wheel" params="name parent radius thickness *origin">
+  <xacro:macro name="wheel" params="name parent radius thickness *origin">
     <link name="${name}_link">
       <inertial>
@@ -37,4 +37,4 @@
       <material>Gazebo/Red</material>
     </gazebo>
-  </macro>
+  </xacro:macro>
 </robot>
